Commit message: Add navigation2 config files

File: botanbot_description/urdf/botanbot.urdf (robot description, URDF)
Before this commit: robot botanbot, 18 links, 17 joints
Links:
- removed link base_scan
- removed link caster_back_link
- removed link caster_front_link
- removed link wheel_left_link
- removed link wheel_right_link
- added link front_left_wheel; collision mesh filename=package://botanbot_description/meshes/wheel.stl scale=1 1 1; visual mesh filename=package://botanbot_description/meshes/wheel.stl scale=1 1 1
- added link front_right_wheel; collision mesh filename=package://botanbot_description/meshes/wheel.stl scale=1 1 1; visual mesh filename=package://botanbot_description/meshes/wheel.stl scale=1 1 1
- added link gps_link; collision mesh filename=package://botanbot_description/meshes/gps.stl scale=0.0005 0.0005 0.001; visual mesh filename=package://botanbot_description/meshes/gps.stl scale=0.0005 0.0005 0.001
- added link rear_axle; collision cylinder length=0.694281 radius=0.043346; visual cylinder length=0.05 radius=0.15
- added link rear_right_wheel; collision mesh filename=package://botanbot_description/meshes/wheel.stl scale=1 1 1; visual mesh filename=package://botanbot_description/meshes/wheel.stl scale=1 1 1
- added link steering_wheel; collision mesh filename=package://botanbot_description/meshes/wheel.stl scale=0.5 0.5 1; visual mesh filename=package://botanbot_description/meshes/wheel.stl scale=0.5 0.5 1
- added link velodyne_link; collision mesh filename=package://botanbot_description/meshes/lidar.stl scale=0.001 0.001 0.001; visual mesh filename=package://botanbot_description/meshes/lidar.stl scale=0.001 0.001 0.001
- link base_link: geometry collision mesh filename=package://botanbot_description/meshes/base.stl; visual mesh filename=package://botanbot_description/meshes/base.stl
- link camera_bottom_screw_frame: geometry collision mesh filename=package://botanbot_description/d435.dae; visual mesh filename=package://botanbot_description/d435.dae
- link imu_link: geometry collision cylinder length=0.011 radius=0.001; visual cylinder length=0.011 radius=0.001
Joints:
- removed joint caster_back_joint
- removed joint caster_front_joint
- removed joint lidar_joint
- removed joint wheel_left_joint
- removed joint wheel_right_joint
- added joint front_left_combined_joint: type continuous, parent base_link, child front_left_wheel, origin xyz=0.653624 0.496194 -0.084805 rpy=0 -0 1.5706, axis 1 0 1
- added joint front_right_combined_joint: type continuous, parent base_link, child front_right_wheel, origin xyz=0.666123 -0.495391 -0.085288 rpy=0 0 1.5706, axis 1 0 1
- added joint gps_joint: type fixed, parent base_link, child gps_link, origin xyz=0 0 0.4 rpy=0 0 0
- added joint rear_left_joint: type continuous, parent base_link, child rear_left_wheel, origin xyz=-0.656583 0.492236 -0.085593 rpy=0 -0 1.5706, axis 1 0 0
- added joint rear_right_joint: type continuous, parent base_link, child rear_right_wheel, origin xyz=-0.644212 -0.499228 -0.085214 rpy=0 -0 1.5706, axis 1 0 0
- added joint steering_joint: type continuous, parent base_link, child steering_wheel, origin xyz=0.400132 9.3e-05 0.399996 rpy=0 -1.57 0, axis 0 0 1
- added joint velodyne_joint: type fixed, parent base_link, child velodyne_link, origin xyz=0 0 0.6 rpy=0 0 0
- joint imu_joint: origin xyz=0 0 0.3 rpy=0 0 0 -> xyz=0.7 0.5 0.6 rpy=0 0 0

Commit message: Add corrections to URDF of botabot_description

File: botanbot_description/urdf/botanbot.urdf (robot description, URDF)
Before this commit: robot botanbot, 20 links, 19 joints
Links:
- added link rear_left_wheel; collision mesh filename=package://botanbot_description/meshes/wheel.stl scale=1 1 1; visual mesh filename=package://botanbot_description/meshes/wheel.stl scale=1 1 1
- link camera_bottom_screw_frame: geometry collision mesh filename=package://botanbot_description/meshes/d435.dae; visual mesh filename=package://botanbot_description/meshes/d435.dae
- link rear_axle: geometry collision cylinder length=0.694281 radius=0.043346; visual cylinder length=0.694281 radius=0.043346
Joints:
- added joint rear_axle_joint: type revolute, parent base_link, child rear_axle, origin xyz=-0.656403 0.001088 -0.085593 rpy=0 0 1.57, axis 0 1 0, limit lower=-0.05 upper=0.05 effort=30 velocity=1.0
- joint base_joint: origin xyz=0 0 0.0 rpy=0 0 0 -> xyz=-0.019375 0.005287 0.340756 rpy=0 0 0
- joint rear_left_joint: parent base_link -> rear_axle
- joint rear_right_joint: parent base_link -> rear_axle

Commit message: set up loal costmap

File: botanbot_description/urdf/botanbot.urdf (robot description, URDF)
Before this commit: robot botanbot, 21 links, 20 joints
Joints:
- joint velodyne_joint: origin xyz=0 0 0.6 rpy=0 0 0 -> xyz=0 0 0.8 rpy=0 0 0

Commit message: configure rbot_ocalization, lgtm for empty GZ wrld

File: botanbot_description/urdf/botanbot.urdf (robot description, URDF)
Before this commit: robot botanbot, 21 links, 20 joints
Links:
- removed link base_footprint
Joints:
- removed joint base_joint
- joint rear_axle_joint: limit lower=-0.05 upper=0.05 effort=30 velocity=1.0 -> lower=-0.05 upper=0.05 effort=0 velocity=0.0

Commit message: fix shaking tf problem

File: botanbot_description/urdf/botanbot.urdf (robot description, URDF)
Before this commit: robot botanbot, 20 links, 19 joints
Joints:
- joint front_left_combined_joint: axis 1 0 1 -> 0 0 1
- joint front_right_combined_joint: axis 1 0 1 -> 0 0 1
- joint rear_axle_joint: type revolute -> continuous
- joint rear_left_joint: parent rear_axle -> base_link
- joint rear_right_joint: parent rear_axle -> base_link

Commit message: test nav2 for outdoor navigation

File: botanbot_description/urdf/botanbot.urdf (robot description, URDF)
Before this commit: robot botanbot, 20 links, 19 joints
Joints:
- joint velodyne_joint: origin xyz=0 0 0.8 rpy=0 0 0 -> xyz=0 0 1.2 rpy=0 0 0

Commit message: Unstable perfromace when converting gps waypoints

File: botanbot_description/urdf/botanbot.urdf (robot description, URDF)
Before this commit: robot botanbot, 20 links, 19 joints
Links:
- removed link gps_link
- added link gps; collision mesh filename=package://botanbot_description/meshes/gps.stl scale=0.0005 0.0005 0.001; visual mesh filename=package://botanbot_description/meshes/gps.stl scale=0.0005 0.0005 0.001
Joints:
- joint gps_joint: child gps_link -> gps

Commit message: test outdoor gps waypoint following

File: botanbot_description/urdf/botanbot.urdf (robot description, URDF)
Before this commit: robot botanbot, 20 links, 19 joints
Joints:
- joint velodyne_joint: origin xyz=0 0 1.2 rpy=0 0 0 -> xyz=0 0 0.9 rpy=0 0 0

Commit message: Add a few corrections for cartogrpaher

File: botanbot_description/urdf/botanbot.urdf (robot description, URDF)
Before this commit: robot botanbot, 20 links, 19 joints
Joints:
- joint imu_joint: origin xyz=0.7 0.5 0.6 rpy=0 0 0 -> xyz=0 0 1.2 rpy=0 0 0

Commit message: support 360 cams, as vSLAM cant cope with turns

File: botanbot_description/urdf/botanbot.urdf (robot description, URDF)
Before this commit: robot botanbot, 20 links, 19 joints
Links:
- added link wide_angle_camera_link
Joints:
- added joint wide_angle_camera_joint: type fixed, parent base_link, child wide_angle_camera_link

Commit message: realsense aint publishing TF :????

File: botanbot_description/urdf/botanbot.urdf (robot description, URDF)
Before this commit: robot botanbot, 21 links, 20 joints
Links:
- link camera_color_frame: geometry collision mesh filename=package://botanbot_description/meshes/d435.dae scale=0.0001 0.0001 0.0001; visual mesh filename=package://botanbot_description/meshes/d435.dae scale=0.0001 0.0001 0.0001
- link camera_color_optical_frame: geometry collision mesh filename=package://botanbot_description/meshes/d435.dae scale=0.0001 0.0001 0.0001; visual mesh filename=package://botanbot_description/meshes/d435.dae scale=0.0001 0.0001 0.0001
- link camera_depth_frame: geometry collision mesh filename=package://botanbot_description/meshes/d435.dae scale=0.0001 0.0001 0.0001; visual mesh filename=package://botanbot_description/meshes/d435.dae scale=0.0001 0.0001 0.0001
- link camera_depth_optical_frame: geometry collision mesh filename=package://botanbot_description/meshes/d435.dae scale=0.0001 0.0001 0.0001; visual mesh filename=package://botanbot_description/meshes/d435.dae scale=0.0001 0.0001 0.0001
- link camera_left_ir_frame: geometry collision mesh filename=package://botanbot_description/meshes/d435.dae scale=0.0001 0.0001 0.0001; visual mesh filename=package://botanbot_description/meshes/d435.dae scale=0.0001 0.0001 0.0001
- link camera_left_ir_optical_frame: geometry collision mesh filename=package://botanbot_description/meshes/d435.dae scale=0.0001 0.0001 0.0001; visual mesh filename=package://botanbot_description/meshes/d435.dae scale=0.0001 0.0001 0.0001
- link camera_link: geometry collision mesh filename=package://botanbot_description/meshes/d435.dae scale=0.0001 0.0001 0.0001; visual mesh filename=package://botanbot_description/meshes/d435.dae scale=0.0001 0.0001 0.0001
- link camera_right_ir_frame: geometry collision mesh filename=package://botanbot_description/meshes/d435.dae scale=0.0001 0.0001 0.0001; visual mesh filename=package://botanbot_description/meshes/d435.dae scale=0.0001 0.0001 0.0001
- link camera_right_ir_optical_frame: geometry collision mesh filename=package://botanbot_description/meshes/d435.dae scale=0.0001 0.0001 0.0001; visual mesh filename=package://botanbot_description/meshes/d435.dae scale=0.0001 0.0001 0.0001
- link wide_angle_camera_link: geometry collision mesh filename=package://botanbot_description/meshes/d435.dae scale=0.0001 0.0001 0.0001; visual mesh filename=package://botanbot_description/meshes/d435.dae scale=0.0001 0.0001 0.0001
