Commit message: finally a wroking version

File: vox_nav_drake_ros/urdf/botanbot.urdf (robot description, URDF)
Before this commit: robot botanbot, 11 links, 11 joints
Links:
- removed link base_footprint
- removed link base_link_0
- removed link base_link_1
- removed link base_link_for_rbt_compat
Joints:
- removed joint base_footprint_joint
- removed joint theta
- removed joint world_joint_for_rbt_compat
- removed joint x
- removed joint y

Commit message: simulate streeing angle too

File: vox_nav_drake_ros/urdf/botanbot.urdf (robot description, URDF)
Before this commit: robot botanbot, 7 links, 6 joints
Joints:
- joint front_left_combined_joint: type continuous -> revolute
- joint front_right_combined_joint: type continuous -> revolute
