Commit message: Use absolute heading from AWSIM imu

File: vox_nav_map_server/urdf/dobbie.urdf (robot description, URDF)
Before this commit: robot dobbie, 7 links, 6 joints
Links:
- removed link sensor_kit_base_link
- added link imu_link; visual cylinder length=0.05 radius=0.05
- added link lidar_link; visual cylinder length=0.05 radius=0.05
Joints:
- added joint imu_link: type fixed, parent base_link, child imu_link, origin xyz=0 0 0.4 rpy=0 0.0 0
- joint lidar_link: child sensor_kit_base_link -> lidar_link

Commit message: update after traversablity estimation experiments

File: vox_nav_map_server/urdf/dobbie.urdf (robot description, URDF)
Before this commit: robot dobbie, 8 links, 7 joints
Links:
- removed link lidar_link
- added link os_sensor; visual cylinder length=0.05 radius=0.05
Joints:
- removed joint lidar_link
- added joint os_sensor: type fixed, parent base_link, child os_sensor, origin xyz=0 0 0.35 rpy=0 0.0 0
